Commit message: 

File: sar_gazebo/models/Source_One/urdf/Source_One.xacro (robot description, xacro)
@@ -305,11 +305,4 @@
   </link>
   <link name="Collision_Radius_Point_Link">
-    <visual>
-        <origin xyz="0 0 0" rpy="0 0 0"/>
-        <geometry>
-          <box size="0.01 0.01 0.01"/>
-        </geometry>
-        <material name="grey"/>
-      </visual>
   </link>
   <joint name="Collision_Radius_Point_Joint" type="fixed">
